File: Prometheus-PRT-1/Prometheus-PRT-1/Prometheus-PRT-1.kicad_pcb (KiCad board)
At the start: 2 copper layers, 64.8 x 7.5 mm, 16 parts, among them J1 Conn_02x10_Odd_Even, J2 AppleIIBus, U1 74LS74, U2 74LS74, U3 74LS00, U4 74LS374, U5 74LS30, U6 74LS08, U7 27C64, U8 74LS08, U9 74LS00

Commit message: Update Prometheus-PRT-1 to kicad8 and the shared symbol library
Parts:
- removed C1, C2: 0.1µ, Capacitor_THT:C_Disc_D4.3mm_W1.9mm_P5.00mm
- removed J1: Conn_02x10_Odd_Even, Connector_PinHeader_2.54mm:PinHeader_2x10_P2.54mm_Vertical
- removed J2: AppleIIBus, Apple:AppleIIBus_Edge
- removed JH1: AckPol, Connector_PinHeader_2.54mm:PinHeader_1x03_P2.54mm_Vertical
- removed JH2: StrobePol, Connector_PinHeader_2.54mm:PinHeader_1x03_P2.54mm_Vertical
- removed R1: 5.5k, Resistor_THT:R_Axial_DIN0207_L6.3mm_D2.5mm_P10.16mm_Horizontal
- removed U1, U2: 74LS74, Package_DIP:DIP-14_W7.62mm_Socket_LongPads
- removed U3, U9: 74LS00, Package_DIP:DIP-14_W7.62mm_Socket_LongPads
- removed U4: 74LS374, Package_DIP:DIP-20_W7.62mm_Socket_LongPads
- removed U5: 74LS30, Package_DIP:DIP-14_W7.62mm_Socket_LongPads
- removed U6, U8: 74LS08, Package_DIP:DIP-14_W7.62mm_Socket_LongPads
- removed U7: 27C64, Package_DIP:DIP-24_W15.24mm
Other:
- board outline removed
