File: Mountain-Computer-CPS-Multifunction-Card/Mountain-Computer-CPS-Multifunction-Card/Mountain-Computer-CPS-Multifunction-Card.kicad_sch (KiCad schematic)
At the start: 51 parts, among them J6 Conn_01x02_Pin, U12 74LS74, U13 74LS273, U14 74LS09, U15 M1-6513H-9, U16 M1-6513H-9, U17 74LS08, U21 74LS123, U22 74LS32, U23 27C16, U24 74LS245, U25 74LS357, U26 74LS32, U3 74LS136, U5 74LS03, U6 74LS138, U7 74LS138, U8 74LS155

Commit message: Update the CPS Multifunction Card
* Found the datasheet for the SRAM being used
* Added a little more information about the mysterious companion board and a workaround to improve stability if you don't have it
* Update the manual quality so it's more legible
Parts:
- removed U15, U16: M1-6513H-9, Package_DIP:DIP-18_W7.62mm, symbol Memory_Legacy:2114
- added U15, U16: HM1-6513H-9, Package_DIP:DIP-18_W7.62mm, symbol Memory_Legacy:HM1-6513H
Connections:
- net +BATT: now also U15.18 (VCC), U16.18 (VCC)
- net GND: now also U15.9 (GND), U16.9 (GND)
- net LD0: now also U15.14 (DQ0)
- net LD1: now also U15.13 (DQ1)
- net LD2: now also U15.12 (DQ2)
- net LD3: now also U15.11 (DQ3)
- net LD4: now also U16.14 (DQ0)
- net LD5: now also U16.13 (DQ1)
- net LD6: now also U16.12 (DQ2)
- net LD7: now also U16.11 (DQ3)
- net RP3_PUP2: now also U16.7 (Y)
- net RP3_PUP5: now also U15.7 (Y)
- net SRAM_BANK0: now also U15.3 (A3), U16.3 (A3)
- net SRAM_BANK1: now also U15.2 (A4), U16.2 (A4)
- net SRAM_BANK2: now also U15.1 (A5), U16.1 (A5)
- net SRAM_BANK3: now also U15.17 (A6), U16.17 (A6)
- net SRAM_BANK4: now also U15.16 (A7), U16.16 (A7)
- net STABLE_A0: now also U15.5 (A1), U16.5 (A1)
- net STABLE_A1: now also U15.6 (A0), U16.6 (A0)
- net STABLE_A2: now also U15.4 (A2), U16.4 (A2)
- net at R8.2, U5.8: now also U15.10 (~{WE}), U16.10 (~{WE})
- net at R7.1, U14.8: now also U15.8 (~{CE}), U16.8 (~{CE})
- net at CR4.1 (K), R9.1: now also U15.15 (A8), U16.15 (A8)
Other:
- note removed: "2114 compatible SRAM?"
- moved on the sheet: C16, CR4, CR5, CR6, J6, R10, R101, R4, R9, U17B, U26C, U5B
