File: Mountain-Computer-CPS-Multifunction-Card/Mountain-Computer-CPS-Multifunction-Card/peripherals.kicad_sch (KiCad schematic)
At the start: 37 parts, among them J1 Conn_01x02_Pin, J2 Conn_01x02_Pin, J3 Conn_01x02_Pin, J4 Conn_02x13_Odd_Even, J5 Conn_02x10_Odd_Even, U1 2651, U10 MSM5832, U11 MC1488, U12 74LS74, U18 74LS173, U19 74LS273, U2 MC1489, U20 74LS367, U21 74LS123, U3 74LS136, U4 74LS374, U9 74LS04, Y1 5.0688 MHz, Y2 32.768 KHz

Commit message: Update the CPS Multifunction Card
* Found the datasheet for the SRAM being used
* Added a little more information about the mysterious companion board and a workaround to improve stability if you don't have it
* Update the manual quality so it's more legible
Other:
- note added: "Top-bottom pin numbering matches what's specified in the manual. This is different than the odd/even numbering used by J5."
- note removed: "Pin numbering matches the manual. The pin ordering is different than J5."
